File: necpc8801l.kicad_sch (KiCad schematic)
At the start: 217 parts, among them J1 Conn_01x04_MountingPin, SW1 SW_Push, U1 ATmega32U4-MU, Y1 16MHz

Commit message: updates
Parts:
- SW_0_1, SW_1_1, SW_2_1, SW_3_1, SW_4_1, SW_5_1, SW_6_1, SW_7_1, SW_8_1, SW_9_1, SW_ALT_1, SW_AMG_1, SW_AT_1, SW_A_1, SW_B_1, SW_CAPS_1, SW_CAR_1, SW_COL_1, SW_CPY_1, SW_CTRL_1, SW_C_1, SW_DEL_1, SW_DOWN_1, SW_D_1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: footprint MX_NEC:MX_NEC -> MX_NEC:mx-nec-alps
